File: optocoupler-shield.sch (EAGLE design)
At the start: 0 parts

Commit message: added optoisolators and config jumpers; jumpers are all connected to shield IO pins
Parts:
- added JP10, JP11, JP8, JP9: M023.5MM, SparkFun-Connectors:M023.5MM
- added JP15: POWER, SmartPrj:PINHD-1X8
- added JP2: PWML, SmartPrj:PINHD-1X8
- added JP3: COMMUNICATION, SmartPrj:PINHD-1X8
- added JP4: XIO, SmartPrj:PINHD-2X18
- added JP5: ADCH, SmartPrj:PINHD-1X8
- added JP6: ADCL, SmartPrj:PINHD-1X8
- added JP7: PWMH, SmartPrj:PINHD-1X10
- added Q1, Q2, Q3, Q4: NPN, SparkFun:TRANSISTOR_NPNSOT23-3
- added R1, R2, R7, R9: 220, SparkFun:RESISTOR0402
- added R10, R11, R12, R3, R4, R5, R6, R8: 10K, SparkFun:RESISTOR0402
- added SPI1: SPI, SmartPrj:PINHD-2X3
- added U$1, U$3, U$4, U$7: PINHD-2X8, headers:PINHD-2X8
- added U$2, U$5, U$6: FIDUCIAL, adafruit:FIDUCIAL
- added U1, U2: OPTO, SparkFun:OPTOISOLATOR-2SOIC8
Connections:
- new net !ADC_RESET_1: JP4.28
- new net AGND: JP4.35, JP4.36, SPI1.6
- new net D38: JP4.19, U$1.1, U$3.1, U$4.1, U$7.1
- new net D39: JP4.20, U$1.3, U$3.3, U$4.3, U$7.3
- new net D40: JP4.21, U$1.5, U$3.5, U$4.5, U$7.5
- new net D41: JP4.22, U$1.7, U$3.7, U$4.7, U$7.7
- new net D42: JP4.23, U$1.9, U$3.9, U$4.9, U$7.9
- new net D43: JP4.24, U$1.11, U$3.11, U$4.11, U$7.11
- new net D44: JP4.25, U$1.13, U$3.13, U$4.13, U$7.13
- new net D45: JP4.26, U$1.15, U$3.15, U$4.15, U$7.15
- new net GND: U1.C1, U1.C2, U2.C1, U2.C2
- new net HV-GND: JP11.1, JP9.1, Q1.E, Q2.E, Q3.E, Q4.E, U1.EM1, U1.EM2, U2.EM1, U2.EM2
- new net IN1: R1.1, U$1.10, U$1.12, U$1.14, U$1.16, U$1.2, U$1.4, U$1.6, U$1.8
- new net IN2: R2.2, U$3.10, U$3.12, U$3.14, U$3.16, U$3.2, U$3.4, U$3.6, U$3.8
- new net IN3: R7.1, U$4.10, U$4.12, U$4.14, U$4.16, U$4.2, U$4.4, U$4.6, U$4.8
- new net IN4: R9.2, U$7.10, U$7.12, U$7.14, U$7.16, U$7.2, U$7.4, U$7.6, U$7.8
- new net N$1: JP7.9
- new net N$10: JP7.6
- new net N$109: JP4.31
- new net N$11: JP7.7
- new net N$110: JP6.6
- new net N$112: JP6.7
- new net N$114: JP15.5
- new net N$115: JP4.1
- new net N$116: JP4.2
- new net N$12: JP7.10
- new net N$13: JP2.1
- new net N$14: JP2.2
- new net N$15: JP2.3
- new net N$16: JP2.5
- new net N$17: JP2.6
- new net N$18: JP2.8
- new net N$19: JP3.1
- new net N$2: JP5.1
- new net N$20: R2.1, U1.A2
- new net N$21: R7.2, U2.A1
- new net N$22: JP3.2
- new net N$23: R9.1, U2.A2
- new net N$25: JP3.5
- new net N$26: JP3.6
- new net N$3: JP15.1
- new net N$32: JP3.8
- new net N$37: JP5.8
- new net N$4: JP3.7
- new net N$43: JP5.7
- new net N$44: JP5.6
- new net N$5: JP2.7
- new net N$55: JP5.5
- new net N$56: JP5.4
- new net N$569: JP6.8
- new net N$57: JP5.3
- new net N$570: JP15.2
- new net N$571: JP15.4
- new net N$572: JP6.1
- new net N$573: JP6.5
- new net N$574: JP7.1
- new net N$575: JP7.2
- new net N$576: JP7.8
- new net N$577: JP2.4
- new net N$578: JP3.3
- new net N$579: JP3.4
- new net N$58: JP5.2
- new net N$580: JP4.5
- new net N$581: JP4.7
- new net N$582: JP4.11
- new net N$583: JP4.13
- new net N$584: JP4.27
- new net N$585: JP4.29
- new net N$586: JP4.33
- new net N$587: JP4.4
- new net N$588: JP4.6
- new net N$589: JP4.8
- new net N$590: JP4.12
- new net N$591: JP4.14
- new net N$592: JP4.30
- new net N$6: R1.2, U1.A1
- new net N$65: JP6.4
- new net N$66: JP6.3
- new net N$68: JP6.2
- new net N$69: JP15.8
- new net N$7: JP7.3
- new net N$70: JP15.7
- new net N$71: JP15.6
- new net N$72: JP15.3
- new net N$73: JP4.34
- new net N$74: JP4.32
- new net N$8: JP7.4
- new net N$89: JP4.18
- new net N$9: JP7.5
- new net N$91: JP4.16
- new net N$92: JP4.10
- new net N$93: JP4.3
- new net N$94: JP4.9
- new net N$96: JP4.15
- new net N$97: JP4.17
- new net OUT1: JP10.2, Q2.C, R6.1
- new net OUT1N: Q2.B, R3.1, U1.CL1
- new net OUT1N1: Q4.B, R8.1, U2.CL1
- new net OUT2: JP11.2, Q1.C, R5.1
- new net OUT2N: Q1.B, R4.1, U1.CL2
- new net OUT2N1: Q3.B, R10.1, U2.CL2
- new net OUT3: JP8.2, Q4.C, R12.1
- new net OUT4: JP9.2, Q3.C, R11.1
- new net RESET: SPI1.5
- new net SPI0_MISO: SPI1.1
- new net SPI0_MOSI: SPI1.4
- new net SPI0_SCK: SPI1.3
- new net VCC: JP10.1, JP8.1, R10.2, R11.2, R12.2, R3.2, R4.2, R5.2, R6.2, R8.2
- new net VCC_5V: SPI1.2
Other:
- note added: "22"
- note added: "23"
- note added: "24"
- note added: "25"
- note added: "26"
- note added: "27"
- note added: "28"
- note added: "29"
- note added: "30"
- note added: "31"
- note added: "32"
- note added: "33"
- note added: "34"
- note added: "35"
- note added: "36"
- note added: "37"
- note added: "38"
- note added: "39"
- note added: "3V to 5V System"
- note added: "3V3"
- note added: "40"
- note added: "41"
- note added: "42"
- note added: "43"
- note added: "44"
- note added: "45"
- note added: "46"
- note added: "47"
- note added: "48"
- note added: "49"
- note added: "50"
- note added: "51"
- note added: "52"
- note added: "53"
- note added: "5V"
- note added: "751-1312-1-ND"
- note added: "A0"
- note added: "A1"
- note added: "A10"
- note added: "A11"
- note added: "A2"
- note added: "A3"
- note added: "A4"
- note added: "A5"
- note added: "A6"
- note added: "A7"
- note added: "A8"
- note added: "A9"
- note added: "AREF"
- note added: "CANRX"
- note added: "CANTX"
- note added: "Configuration jumpers"
- note added: "Copyright 2013 Adam Feuer"
- note added: "D0"
- note added: "D1"
- note added: "D10"
- note added: "D11"
- note added: "D12"
- note added: "D13"
- note added: "D14"
- note added: "D15"
- note added: "D16"
- note added: "D17"
- note added: "D18"
- note added: "D19"
- note added: "D2"
- note added: "D20"
- note added: "D21"
- note added: "D3"
- note added: "D4"
- note added: "D5"
- note added: "D6"
- note added: "D7"
- note added: "D8"
- note added: "D9"
- note added: "DAC0"
- note added: "DAC1"
- note added: "Fiducials (for pick and place machines)"
- note added: "GND"
- note added: "ILD213T"
- note added: "IOREF"
- note added: "NOT USED"
- note added: "Noisy System"
- note added: "Pins not labeled are not connected (NC)"
- note added: "RESET"
- note added: "RX2"
- note added: "Released under a Creative Commons By-Attribution Share-Alike 3.0 license"
- note added: "SCL1"
- note added: "SDA1"
- note added: "Shield Connectors"
- note added: "TX2"
- note added: "VIN"
