File: optoisolator-shield.sch (EAGLE design)
At the start: 37 parts, among them Q1 NPN, Q2 NPN, Q3 NPN, Q4 NPN, U1 OPTO, U2 OPTO

Commit message: fixed direction of optoisolators; added an output to go along with the 2 inputs; all components are still SMT
Parts:
- removed JP11: M023.5MM, SparkFun-Connectors:M023.5MM
- removed U$1, U$3, U$4, U$7: PINHD-2X8, headers:PINHD-2X8
- added INPUT1, INPUT2, INPUT3, INPUT4, OUTPUT1, OUTPUT2: PINHD-2X8, headers:PINHD-2X8
- added JP1: (no value), SparkFun-Connectors:M03SCREW
- added Q5, Q6: NPN, SparkFun:TRANSISTOR_NPNSOT23-3
- added R13, R15: 220, SparkFun:RESISTOR0402
- added R14, R16, R17, R18: 10K, SparkFun:RESISTOR0402
- added U3: OPTO, SparkFun:OPTOISOLATOR-2SOIC8
- JP8: value M023.5MM -> (none); device SparkFun-Connectors:M023.5MM -> SparkFun-Connectors:M03SCREW
- R2: value 220 -> 10K
- R3: value 10K -> 220
Connections:
- net OUT2N renamed OUT2N2
- removed net HV-GND: JP11.1, JP9.1, Q1.E, Q2.E, Q3.E, Q4.E, U1.EM1, U1.EM2, U2.EM1, U2.EM2
- removed net N$570: JP15.2
- removed net N$70: JP15.7
- removed net OUT1: JP10.2, Q2.C, R6.1
- removed net OUT1N: Q2.B, R3.1, U1.CL1
- removed net OUT2: JP11.2, Q1.C, R5.1
- removed net OUT3: JP8.2, Q4.C, R12.1
- removed net OUT4: JP9.2, Q3.C, R11.1
- new net EXT_GND_0: JP8.1, U1.C1, U1.C2
- new net EXT_GND_1: JP1.1, U2.C1, U2.C2
- new net EXT_GND_2: JP10.1, Q5.E, Q6.E, U3.EM1, U3.EM2
- new net EXT_VCC: JP9.1, R14.2, R16.2, R17.2, R18.2
- new net IN6: OUTPUT2.10, OUTPUT2.12, OUTPUT2.14, OUTPUT2.16, OUTPUT2.2, OUTPUT2.4, OUTPUT2.6, OUTPUT2.8
- new net N$24: R13.2, U3.A1
- new net N$27: R15.1, U3.A2
- new net OPTO_IN5: OUTPUT1.10, OUTPUT1.12, OUTPUT1.14, OUTPUT1.16, OUTPUT1.2, OUTPUT1.4, OUTPUT1.6, OUTPUT1.8, R13.1
- new net OPTO_IN6: R15.2
- new net OPTO_OUT1: INPUT1.10, INPUT1.12, INPUT1.14, INPUT1.16, INPUT1.2, INPUT1.4, INPUT1.6, INPUT1.8, Q2.C, R6.1
- new net OPTO_OUT2: INPUT2.10, INPUT2.12, INPUT2.14, INPUT2.16, INPUT2.2, INPUT2.4, INPUT2.6, INPUT2.8, Q1.C, R5.1
- new net OPTO_OUT3: INPUT3.10, INPUT3.12, INPUT3.14, INPUT3.16, INPUT3.2, INPUT3.4, INPUT3.6, INPUT3.8, Q4.C, R12.1
- new net OPTO_OUT4: INPUT4.10, INPUT4.12, INPUT4.14, INPUT4.16, INPUT4.2, INPUT4.4, INPUT4.6, INPUT4.8, Q3.C, R11.1
- new net OUT1N2: Q2.B, R2.1, U1.CL1
- new net OUT1N3: Q6.B, R14.1, U3.CL1
- new net OUT2N3: Q5.B, R16.1, U3.CL2
- new net OUT5: Q6.C, R18.1
- new net OUT6: Q5.C, R17.1
- net D38: now also INPUT1.1, INPUT2.1, INPUT3.1, INPUT4.1, OUTPUT1.1, OUTPUT2.1; no longer U$1.1, U$3.1, U$4.1, U$7.1
- net D39: now also INPUT1.3, INPUT2.3, INPUT3.3, INPUT4.3, OUTPUT1.3, OUTPUT2.3; no longer U$1.3, U$3.3, U$4.3, U$7.3
- net D40: now also INPUT1.5, INPUT2.5, INPUT3.5, INPUT4.5, OUTPUT1.5, OUTPUT2.5; no longer U$1.5, U$3.5, U$4.5, U$7.5
- net D41: now also INPUT1.7, INPUT2.7, INPUT3.7, INPUT4.7, OUTPUT1.7, OUTPUT2.7; no longer U$1.7, U$3.7, U$4.7, U$7.7
- net D42: now also INPUT1.9, INPUT2.9, INPUT3.9, INPUT4.9, OUTPUT1.9, OUTPUT2.9; no longer U$1.9, U$3.9, U$4.9, U$7.9
- net D43: now also INPUT1.11, INPUT2.11, INPUT3.11, INPUT4.11, OUTPUT1.11, OUTPUT2.11; no longer U$1.11, U$3.11, U$4.11, U$7.11
- net D44: now also INPUT1.13, INPUT2.13, INPUT3.13, INPUT4.13, OUTPUT1.13, OUTPUT2.13; no longer U$1.13, U$3.13, U$4.13, U$7.13
- net D45: now also INPUT1.15, INPUT2.15, INPUT3.15, INPUT4.15, OUTPUT1.15, OUTPUT2.15; no longer U$1.15, U$3.15, U$4.15, U$7.15
- net GND: now also JP15.7, Q1.E, Q2.E, Q3.E, Q4.E, U1.EM1, U1.EM2, U2.EM1, U2.EM2, U3.C1, U3.C2; no longer U1.C1, U1.C2, U2.C1, U2.C2
- net IN1: now also JP8.3; no longer U$1.10, U$1.12, U$1.14, U$1.16, U$1.2, U$1.4, U$1.6, U$1.8
- net IN2: now also JP8.2, R3.2; no longer R2.2, U$3.10, U$3.12, U$3.14, U$3.16, U$3.2, U$3.4, U$3.6, U$3.8
- net IN3: now also JP1.3; no longer U$4.10, U$4.12, U$4.14, U$4.16, U$4.2, U$4.4, U$4.6, U$4.8
- net IN4: now also JP1.2; no longer U$7.10, U$7.12, U$7.14, U$7.16, U$7.2, U$7.4, U$7.6, U$7.8
- net N$20: now also R3.1; no longer R2.1
- net VCC: now also JP15.2, R2.2; no longer JP10.1, JP8.1, R3.2
Other:
- note added: "Arduino"
- note added: "External (noisy) system"
- note added: "Input (External to Arduino)"
- note added: "Output (Arduino to External)"
- note removed: "3V to 5V System"
- note removed: "751-1312-1-ND"
- note removed: "Noisy System"
- moved on the sheet: JP10, JP9, Q1, Q2, Q3, Q4, R1, R10, R11, R12, R2, R3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
